File: temp.sensor/pcb/board.brd (EAGLE design)
At the start: 68.1 x 31.4 mm, 13 parts, among them IC1 BME280

Commit message: ddd
Parts:
- added C1: (no value), rcl:E1,8-4
- added Q1, Q2: BC849SMD, transistor-npn:SOT23-BEC
- added R5, R6: (no value), rcl:R1206
- JP1: device pinhead:1X04/90 -> pinhead:1X06/90
- R1: device rcl:0207/10 -> rcl:R1206
- moved R1 2.39 mm to (15.6, 21.4)
- moved R2 1.77 mm to (15.6, 1.91)
- moved IC1 1.11 mm to (11.4, 15.7)
- moved JP1 0.85 mm to (6.51, 7.94)
- moved X3 0.32 mm to (62.7, 25.7)
- renumbered SJR1 to ESP12, U$1 to .., U$2 to .
Connections:
- new net DTR: JP1.6, Q2.E, R5.1
- new net N$3: Q1.B, R5.2
- new net N$4: Q2.B, R6.2
- new net R/C: JP1.2, Q1.E, R6.1
- net 3V3: now also C1.+, JP1.3; no longer JP1.1
- net GND: now also C1.-, JP1.1; no longer JP1.2
- net GPIO0: now also Q2.C
- net RST: now also Q1.C
- net RX: now also JP1.4; no longer JP1.3
- net TX: now also JP1.5; no longer JP1.4
Routing:
- net RST: track 37.9 -> 52.1 mm
- net DTR: track 0.00 -> 4.49 mm
- net GND: track 8.50 -> 12.4 mm
- net R/C: track 0.00 -> 2.47 mm
- net GPIO0: track 66.4 -> 67.2 mm
- net GPIO15: track 4.41 -> 3.67 mm
- net SDA: track 20.1 -> 20.8 mm
Other:
- board text added: "+"
- board text added: "^-"
