File: temp.sensor/pcb/board.sch (EAGLE design)
At the start: 13 parts, among them IC1 BME280

Commit message: ddd
Parts:
- added C1: (no value), rcl:CPOL-EUE1.8-4
- added Q1, Q2: BC849SMD, transistor-npn:BC849SMD
- added R5, R6: (no value), rcl:R-EU_R1206
- JP1: device pinhead:PINHD-1X4/90 -> pinhead:PINHD-1X6/90
- R1: device rcl:R-EU_0207/10 -> rcl:R-EU_R1206
- renumbered SJR1 to ESP12, U$1 to .., U$2 to .
Connections:
- new net DTR: JP1.6, Q2.E, R5.1
- new net N$3: Q1.B, R5.2
- new net N$4: Q2.B, R6.2
- new net R/C: JP1.2, Q1.E, R6.1
- net 3V3: now also C1.+, JP1.3; no longer JP1.1
- net GND: now also C1.-, JP1.1; no longer JP1.2
- net GPIO0: now also Q2.C
- net RST: now also Q1.C
- net RX: now also JP1.4; no longer JP1.3
- net TX: now also JP1.5; no longer JP1.4
