File: stove.regulator/pcb/untitled1.brd (EAGLE design)
At the start: 78.1 x 56.8 mm, 10 parts, among them IC1 4051N

Commit message: part of config
Parts:
- added IC2: 4051N, 40xx:DIL16
- added JP5: (no value), pinhead:1X04
- added JP6, JP7, JP8: (no value), pinhead:1X02
- added R2: (no value), rcl:0207/10
- added U$1: HLK-PM01, diy-modules:HLK-PM01
- added WEMOS2: (no value), esp8266modules:WEMOS-D1-MINI
- added X3, X4: (no value), con-wago-500:W237-102
- moved JP3 1.91 mm to (72.4, 14.6)
- moved JP2 1.59 mm to (72.4, 6.99)
- moved JP4 1.59 mm to (72.4, 21.9)
Connections:
- new net 3V1: IC2.16, JP5.3, JP6.2, JP7.2, JP8.2, WEMOS2.3V3
- new net 5V1: U$1.P$4, WEMOS2.5V
- new net D1: IC2.9, WEMOS2.D8
- new net D2: IC2.10, WEMOS2.D7
- new net D3: IC2.11, WEMOS2.D6
- new net GND1: IC2.6, IC2.7, IC2.8, JP5.4, R2.2, U$1.P$3, X4.1
- new net N$10: IC2.3, R2.1, WEMOS2.A0
- new net N$11: IC2.13, JP8.1
- new net N$12: IC2.14, JP7.1
- new net N$13: IC2.15, JP6.1
- new net N$14: JP5.1, WEMOS2.D2
- new net N$15: JP5.2, WEMOS2.D1
- new net N$16: U$1.P$1, X3.1
- new net N$17: U$1.P$2, X3.2
- new net N$18: WEMOS2.D3, X4.2
- net GND: no longer WEMOS1.GND
Routing:
- net 3V1: track 0.00 -> 134.9 mm
- net N$15: track 0.00 -> 86.6 mm
- net N$14: track 0.00 -> 81.9 mm
- net N$18: track 0.00 -> 57.4 mm, vias 0 -> 2
- net 5V1: track 0.00 -> 46.9 mm
- net N$6: track 47.9 -> 86.6 mm
- net N$5: track 45.7 -> 81.9 mm
- net N$10: track 0.00 -> 34.6 mm
- net N$13: track 0.00 -> 29.8 mm
- net N$16: track 0.00 -> 26.3 mm
- net N$11: track 0.00 -> 23.0 mm
- net N$12: track 0.00 -> 22.1 mm
- net N$17: track 0.00 -> 11.0 mm
- net 3V3: track 126.3 -> 134.9 mm
- net D1: track 0.00 -> 7.19 mm
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- added copper zone on layer 16, net GND1
Other:
- board size 78.1 x 56.8 mm -> 78.1 x 116.8 mm
